Commit message: created plug, added to D415

File: realsense2_description/urdf/_d415.urdf.xacro (robot description, xacro)
@@ -9,5 +9,6 @@
   <!-- Includes -->
   <xacro:include filename="$(find realsense2_description)/urdf/_materials.urdf.xacro" />
-  <xacro:macro name="sensor_d415" params="parent *origin  name:=camera  use_nominal_extrinsics:=false">
+  <xacro:include filename="$(find realsense2_description)/urdf/_usb_plug.urdf.xacro" />
+  <xacro:macro name="sensor_d415" params="parent *origin  name:=camera  use_nominal_extrinsics:=false  add_plug:=false">
     <xacro:property name="M_PI" value="3.1415926535897931" />
     <!-- The following values are approximate, and the camera node
@@ -117,4 +118,9 @@
       <link name="${name}_color_optical_frame"/>
     </xacro:if>
+    <xacro:if value="$(arg add_plug)">
+      <xacro:usb_plug parent="${name}_link">
+        <origin xyz="${d415_cam_mount_from_center_offset - 0.01587} ${-d415_cam_depth_py - 0.0358} 0" rpy="0 0 0"/>
+      </xacro:usb_plug>
+    </xacro:if>
   </xacro:macro>
 </robot>

Commit message: D435 too

File: realsense2_description/urdf/_d415.urdf.xacro (robot description, xacro)
@@ -3,5 +3,5 @@
 License: Apache 2.0. See LICENSE file in root directory.
 Copyright(c) 2017 Intel Corporation. All Rights Reserved
-This is the URDF model for the Intel RealSense 415 camera, in it's
+This is the URDF model for the Intel RealSense 415 camera, in its
 aluminum peripherial evaluation case.
 -->

File: realsense2_description/urdf/_d435.urdf.xacro (robot description, xacro)
@@ -3,5 +3,5 @@
 License: Apache 2.0. See LICENSE file in root directory.
 Copyright(c) 2017 Intel Corporation. All Rights Reserved
-This is the URDF model for the Intel RealSense 430 camera, in it's
+This is the URDF model for the Intel RealSense 430 camera, in its
 aluminum peripherial evaluation case.
 -->
@@ -9,4 +9,5 @@
   <!-- Includes -->
   <xacro:include filename="$(find realsense2_description)/urdf/_materials.urdf.xacro" />
+  <xacro:include filename="$(find realsense2_description)/urdf/_usb_plug.urdf.xacro" />
   <xacro:macro name="sensor_d435" params="parent *origin name:=camera use_nominal_extrinsics:=false">
     <xacro:property name="M_PI" value="3.1415926535897931" />
@@ -116,4 +117,9 @@
       <link name="${name}_color_optical_frame"/>
     </xacro:if>
+    <xacro:if value="$(arg add_plug)">
+      <xacro:usb_plug parent="${name}_link">
+        <origin xyz="${d435_cam_mount_from_center_offset - 0.02095} ${-d435_cam_depth_py - 0.0353} 0" rpy="0 0 0"/>
+      </xacro:usb_plug>
+    </xacro:if>
   </xacro:macro>
 </robot>

Commit message: commented out the material from the included materials file (aluminum) and added it with the name suffix to the camera urdf.

File: realsense2_description/urdf/_d415.urdf.xacro (robot description, xacro)
@@ -8,5 +8,5 @@
 <robot name="sensor_d415" xmlns:xacro="http://ros.org/wiki/xacro">
   <!-- Includes -->
-  <xacro:include filename="$(find realsense2_description)/urdf/_materials.urdf.xacro" />
+  <!-- <xacro:include filename="$(find realsense2_description)/urdf/_materials.urdf.xacro" /> -->
   <xacro:macro name="sensor_d415" params="parent *origin  name:=camera  use_nominal_extrinsics:=false">
     <xacro:property name="M_PI" value="3.1415926535897931" />
@@ -28,4 +28,7 @@
     <xacro:property name="d415_cam_depth_py" value="0.020"/>
     <xacro:property name="d415_cam_depth_pz" value="${d415_cam_height/2}"/>
+    <material name="${name}_aluminum">
+	    <color rgba="0.5 0.5 0.5 1"/>
+    </material>
     <!-- camera body, with origin at bottom screw mount -->
     <joint name="${name}_joint" type="fixed">

File: realsense2_description/urdf/_d435.urdf.xacro (robot description, xacro)
@@ -8,5 +8,5 @@
 <robot name="sensor_d435" xmlns:xacro="http://ros.org/wiki/xacro">
   <!-- Includes -->
-  <xacro:include filename="$(find realsense2_description)/urdf/_materials.urdf.xacro" />
+  <!-- <xacro:include filename="$(find realsense2_description)/urdf/_materials.urdf.xacro" /> -->
   <xacro:macro name="sensor_d435" params="parent *origin name:=camera use_nominal_extrinsics:=false">
     <xacro:property name="M_PI" value="3.1415926535897931" />
@@ -28,4 +28,7 @@
     <xacro:property name="d435_cam_depth_py" value="0.0175"/>
     <xacro:property name="d435_cam_depth_pz" value="${d435_cam_height/2}"/>
+    <material name="${name}_aluminum">
+	    <color rgba="0.5 0.5 0.5 1"/>
+    </material>
     <!-- camera body, with origin at bottom screw mount -->
     <joint name="${name}_joint" type="fixed">

File: realsense2_description/urdf/_r410.urdf.xacro (robot description, xacro)
@@ -8,5 +8,5 @@
 <robot name="sensor_r410" xmlns:xacro="http://ros.org/wiki/xacro">
   <!-- Includes -->
-  <xacro:include filename="$(find realsense2_description)/urdf/_materials.urdf.xacro" />
+  <!-- <xacro:include filename="$(find realsense2_description)/urdf/_materials.urdf.xacro" /> -->
   <xacro:macro name="sensor_r410" params="parent *origin  name:=camera  use_nominal_extrinsics:=false">
     <xacro:property name="M_PI" value="3.1415926535897931" />
@@ -27,4 +27,7 @@
     <xacro:property name="r410_cam_depth_py" value="-0.0425"/>
     <xacro:property name="r410_cam_depth_pz" value="0.026"/>
+    <material name="${name}_aluminum">
+	    <color rgba="0.5 0.5 0.5 1"/>
+    </material>
     <!-- camera body, with origin at bottom screw mount -->
     <joint name="${name}_joint" type="fixed">

File: realsense2_description/urdf/_r430.urdf.xacro (robot description, xacro)
@@ -8,5 +8,5 @@
 <robot name="sensor_r430" xmlns:xacro="http://ros.org/wiki/xacro">
   <!-- Includes -->
-  <xacro:include filename="$(find realsense2_description)/urdf/_materials.urdf.xacro" />
+  <!-- <xacro:include filename="$(find realsense2_description)/urdf/_materials.urdf.xacro" /> -->
   <xacro:macro name="sensor_r430" params="parent *origin name:=camera use_nominal_extrinsics:=false">
   <xacro:property name="M_PI" value="3.1415926535897931" />
@@ -28,4 +28,7 @@
   <xacro:property name="r430_cam_depth_py" value="-0.035"/>
   <xacro:property name="r430_cam_depth_pz" value="0.028"/>
+  <material name="${name}_aluminum">
+	    <color rgba="0.5 0.5 0.5 1"/>
+  </material>
     <!-- camera body, with origin at bottom screw mount -->
     <joint name="${name}_joint" type="fixed">

Commit message: Consistent add_plug in xacros and launch files

File: realsense2_description/urdf/_d415.urdf.xacro (robot description, xacro)
@@ -10,5 +10,5 @@
   <xacro:include filename="$(find realsense2_description)/urdf/_materials.urdf.xacro" />
   <xacro:include filename="$(find realsense2_description)/urdf/_usb_plug.urdf.xacro" />
-  <xacro:macro name="sensor_d415" params="parent *origin  name:=camera  use_nominal_extrinsics:=false  add_plug:=false">
+  <xacro:macro name="sensor_d415" params="parent *origin  name:=camera  use_nominal_extrinsics:=false add_plug:=false">
     <xacro:property name="M_PI" value="3.1415926535897931" />
     <!-- The following values are approximate, and the camera node

Commit message: Merge branch 'd415_add_plug' of https://github.com/Tuebel/realsense-ros into Tuebel-d415_add_plug
(cherry picked from commit 350ef7029a485cffe46a05935f71fa25fc96c3aa)

File: realsense2_description/urdf/_d415.urdf.xacro (robot description, xacro)
@@ -10,5 +10,5 @@
   <xacro:include filename="$(find realsense2_description)/urdf/_materials.urdf.xacro" />
   <xacro:include filename="$(find realsense2_description)/urdf/_usb_plug.urdf.xacro" />
-  <xacro:macro name="sensor_d415" params="parent *origin  name:=camera  use_nominal_extrinsics:=false  add_plug:=false">
+  <xacro:macro name="sensor_d415" params="parent *origin  name:=camera  use_nominal_extrinsics:=false add_plug:=false">
     <xacro:property name="M_PI" value="3.1415926535897931" />
     <!-- The following values are approximate, and the camera node
@@ -118,5 +118,5 @@
       <link name="${name}_color_optical_frame"/>
     </xacro:if>
-    <xacro:if value="$(arg add_plug)">
+    <xacro:if value="${add_plug}">
       <xacro:usb_plug parent="${name}_link" name="${name}_usb_plug">
         <origin xyz="${d415_cam_mount_from_center_offset - 0.01587} ${-d415_cam_depth_py - 0.0358} 0" rpy="0 0 0"/>

Commit message: fix d415 mass in _d415.urdf.xacro.
import tests for xacro files.

File: realsense2_description/urdf/_d415.urdf.xacro (robot description, xacro)
@@ -57,6 +57,6 @@
       </collision>
       <inertial>
+        <mass value="0.072" />
         <!-- The following are not reliable values, and should not be used for modeling -->
-        <mass value="0.564" />
         <origin xyz="0 0 0" />
         <inertia ixx="0.003881243" ixy="0.0" ixz="0.0" iyy="0.000498940" iyz="0.0" izz="0.003879257" />
