Commit message: Update numbers for d455, use box for vis, add IMU extrinsics

File: realsense2_description/urdf/_d455.urdf.xacro (robot description, xacro)
@@ -16,23 +16,20 @@
      publishing TF values with actual calibrated camera extrinsic values -->
     <xacro:property name="d455_cam_depth_to_infra1_offset" value="0.0"/>
-    <xacro:property name="d455_cam_depth_to_infra2_offset" value="-0.050"/>
-    <xacro:property name="d455_cam_depth_to_color_offset" value="0.015"/>
+    <xacro:property name="d455_cam_depth_to_infra2_offset" value="-0.095"/>
+    <xacro:property name="d455_cam_depth_to_color_offset" value="-0.059"/>
+    <!-- see datasheet Revision 009, Fig. 4-4 page 68 -->
+    <xacro:property name="d455_zero_depth_to_glass" value="4.55e-3"/>
     <!-- The following values model the aluminum peripherial case for the
   	d455 camera, with the camera joint represented by the actual
   	peripherial camera tripod mount -->
-    <xacro:property name="d455_cam_width" value="0.090"/>
-    <xacro:property name="d455_cam_height" value="0.025"/>
-    <xacro:property name="d455_cam_depth" value="0.02505"/>
-    <xacro:property name="d455_cam_mount_from_center_offset" value="0.0149"/>
-    <!-- glass cover is 0.1 mm inwards from front aluminium plate -->
-    <xacro:property name="d455_glass_to_front" value="0.1e-3"/>
-    <!-- see datasheet Revision 007, Fig. 4-4 page 65 -->
-    <xacro:property name="d455_zero_depth_to_glass" value="4.2e-3"/>
-    <!-- convenience precomputation to avoid clutter-->
-    <xacro:property name="d455_mesh_x_offset" value="${d455_cam_mount_from_center_offset-d455_glass_to_front-d455_zero_depth_to_glass}"/>
+    <xacro:property name="d455_cam_width" value="0.124"/>
+    <xacro:property name="d455_cam_height" value="0.029"/>
+    <xacro:property name="d455_cam_depth" value="0.026"/>
+    <xacro:property name="d455_cam_mount_to_front" value="0.0158"/>
+    <xacro:property name="d455_cam_mount_from_center_offset" value="${d455_cam_mount_to_front-d455_zero_depth_to_glass}"/>
     <!-- The following offset is relative the the physical d455 camera peripherial
   	camera tripod mount -->
     <xacro:property name="d455_cam_depth_px" value="${d455_cam_mount_from_center_offset}"/>
-    <xacro:property name="d455_cam_depth_py" value="0.0175"/>
+    <xacro:property name="d455_cam_depth_py" value="0.0475"/>
     <xacro:property name="d455_cam_depth_pz" value="${d455_cam_height/2}"/>
     <!-- camera body, with origin at bottom screw mount -->
@@ -44,5 +41,5 @@
     <link name="${name}_bottom_screw_frame"/>
     <joint name="${name}_link_joint" type="fixed">
-      <origin xyz="${d455_mesh_x_offset} ${d455_cam_depth_py} ${d455_cam_depth_pz}" rpy="0 0 0"/>
+      <origin xyz="${d455_cam_depth_px} ${d455_cam_depth_py} ${d455_cam_depth_pz}" rpy="0 0 0"/>
       <parent link="${name}_bottom_screw_frame"/>
       <child link="${name}_link" />
@@ -50,9 +47,10 @@
     <link name="${name}_link">
       <visual>
+        <origin xyz="0 ${-d455_cam_depth_py} 0" rpy="0 0 0"/>
         <!-- the mesh origin is at front plate in between the two infrared camera axes -->
-        <origin xyz="${d455_zero_depth_to_glass + d455_glass_to_front} ${-d455_cam_depth_py} 0" rpy="${M_PI/2} 0 ${M_PI/2}"/>
+        <!-- <origin xyz="${d455_zero_depth_to_glass + d455_glass_to_front} ${-d455_cam_depth_py} 0" rpy="${M_PI/2} 0 ${M_PI/2}"/> -->
         <geometry>
-          <!-- <box size="${d455_cam_width} ${d455_cam_height} ${d455_cam_depth}"/> -->
-	        <mesh filename="package://realsense2_description/meshes/d455.dae" />
+          <box size="${d455_cam_width} ${d455_cam_height} ${d455_cam_depth}"/>
+	        <!-- <mesh filename="package://realsense2_description/meshes/d455.dae" /> -->
         </geometry>
       </visual>
@@ -124,8 +122,37 @@
       </joint>
       <link name="${name}_color_optical_frame"/>
+      <!-- IMU -->
+      <!-- see datasheet Revision 009, page 114 -->
+      <xacro:property name="d455_imu_px" value="${d455_cam_depth_px-0.01602}"/>
+      <xacro:property name="d455_imu_py" value="0.d455_cam_depth_py-0.03022"/>
+      <xacro:property name="d455_imu_pz" value="${d455_cam_depth_pz+0.0074}"/>
+      <link name="${name}_accel_frame" />
+      <link name="${name}_accel_optical_frame" />
+      <link name="${name}_gyro_frame" />
+      <link name="${name}_gyro_optical_frame" />
+      <joint name="${name}_accel_joint" type="fixed">
+        <origin xyz = "${d455_imu_px} ${d455_imu_py} ${d455_imu_pz}" rpy = "0 0 0" />
+        <parent link="${name}_link" />
+        <child link="${name}_accel_frame" />
+      </joint>
+      <joint name="${name}_accel_optical_joint" type="fixed">
+        <origin xyz = "0 0 0" rpy = "${-M_PI/2} 0 ${-M_PI/2}" />
+        <parent link="${name}_accel_frame" />
+        <child link="${name}_accel_optical_frame" />
+      </joint>
+      <joint name="${name}_gyro_joint" type="fixed">
+        <origin xyz = "${d455_imu_px} ${d455_imu_py} ${d455_imu_pz}" rpy = "0 0 0" />
+        <parent link="${name}_link" />
+        <child link="${name}_gyro_frame" />
+      </joint>
+      <joint name="${name}_gyro_optical_joint" type="fixed">
+        <origin xyz = "0 0 0" rpy = "${-M_PI/2} 0 ${-M_PI/2}" />
+        <parent link="${name}_gyro_frame" />
+        <child link="${name}_gyro_optical_frame" />
+      </joint>
     </xacro:if>
     <xacro:if value="$(arg add_plug)">
       <xacro:usb_plug parent="${name}_link" name="${name}_usb_plug">
-        <origin xyz="${d455_cam_mount_from_center_offset - 0.02095} ${-d455_cam_depth_py - 0.0353} 0" rpy="0 0 0"/>
+        <origin xyz="-0.00406 0.03701 0" rpy="0 ${-M_PI/2} 0"/>
       </xacro:usb_plug>
     </xacro:if>

Commit message: Fix D455 urdf

File: realsense2_description/urdf/_d455.urdf.xacro (robot description, xacro)
@@ -51,5 +51,5 @@
         <!-- <origin xyz="${d455_zero_depth_to_glass + d455_glass_to_front} ${-d455_cam_depth_py} 0" rpy="${M_PI/2} 0 ${M_PI/2}"/> -->
         <geometry>
-          <box size="${d455_cam_width} ${d455_cam_height} ${d455_cam_depth}"/>
+          <box size="${d455_cam_depth} ${d455_cam_width} ${d455_cam_height}"/>
 	        <!-- <mesh filename="package://realsense2_description/meshes/d455.dae" /> -->
         </geometry>
@@ -124,7 +124,7 @@
       <!-- IMU -->
       <!-- see datasheet Revision 009, page 114 -->
-      <xacro:property name="d455_imu_px" value="${d455_cam_depth_px-0.01602}"/>
-      <xacro:property name="d455_imu_py" value="0.d455_cam_depth_py-0.03022"/>
-      <xacro:property name="d455_imu_pz" value="${d455_cam_depth_pz+0.0074}"/>
+      <xacro:property name="d455_imu_px" value="-0.01602"/>
+      <xacro:property name="d455_imu_py" value="-0.03022"/>
+      <xacro:property name="d455_imu_pz" value="+0.0074"/>
       <link name="${name}_accel_frame" />
       <link name="${name}_accel_optical_frame" />

Commit message: Fix D455 box location

File: realsense2_description/urdf/_d455.urdf.xacro (robot description, xacro)
@@ -47,5 +47,5 @@
     <link name="${name}_link">
       <visual>
-        <origin xyz="0 ${-d455_cam_depth_py} 0" rpy="0 0 0"/>
+        <origin xyz="${d455_zero_depth_to_glass-d455_cam_depth/2} ${-d455_cam_depth_py} 0" rpy="0 0 0"/>
         <!-- the mesh origin is at front plate in between the two infrared camera axes -->
         <!-- <origin xyz="${d455_zero_depth_to_glass + d455_glass_to_front} ${-d455_cam_depth_py} 0" rpy="${M_PI/2} 0 ${M_PI/2}"/> -->
@@ -56,5 +56,5 @@
       </visual>
       <collision>
-        <origin xyz="0 ${-d455_cam_depth_py} 0" rpy="0 0 0"/>
+        <origin xyz="${d455_zero_depth_to_glass-d455_cam_depth/2} ${-d455_cam_depth_py} 0" rpy="0 0 0"/>
         <geometry>
           <box size="${d455_cam_depth} ${d455_cam_width} ${d455_cam_height}"/>

Commit message: Fix sign of D455 plug y offset

File: realsense2_description/urdf/_d455.urdf.xacro (robot description, xacro)
@@ -154,5 +154,5 @@
     <xacro:if value="$(arg add_plug)">
       <xacro:usb_plug parent="${name}_link" name="${name}_usb_plug">
-        <origin xyz="-0.00406 0.03701 0" rpy="0 ${-M_PI/2} 0"/>
+        <origin xyz="${-0.00406-d455_cam_depth_px} ${-0.03701-d455_cam_depth_py} ${-d455_cam_depth_pz}" rpy="${M_PI/2} 0 0"/>
       </xacro:usb_plug>
     </xacro:if>

Commit message: Add d455 mesh
Mesh used from https://github.com/felixvd/realsense-ros/blob/development/realsense2_description/meshes/d455.stl
Scale and position copied from https://github.com/felixvd/realsense-ros/blob/development/realsense2_description/urdf/_d455.urdf.xacro

File: realsense2_description/urdf/_d455.urdf.xacro (robot description, xacro)
@@ -47,10 +47,10 @@
     <link name="${name}_link">
       <visual>
-        <origin xyz="${d455_zero_depth_to_glass-d455_cam_depth/2} ${-d455_cam_depth_py} 0" rpy="0 0 0"/>
         <!-- the mesh origin is at front plate in between the two infrared camera axes -->
-        <!-- <origin xyz="${d455_zero_depth_to_glass + d455_glass_to_front} ${-d455_cam_depth_py} 0" rpy="${M_PI/2} 0 ${M_PI/2}"/> -->
+        <!-- <origin xyz="${d455_zero_depth_to_glass-d455_cam_depth/2} ${-d455_cam_depth_py} 0" rpy="0 0 0"/> -->
+        <origin xyz="${0} ${-d455_cam_depth_py} 0" rpy="${M_PI/2} 0 ${M_PI/2}"/>
         <geometry>
-          <box size="${d455_cam_depth} ${d455_cam_width} ${d455_cam_height}"/>
-	        <!-- <mesh filename="package://realsense2_description/meshes/d455.dae" /> -->
+          <!-- <box size="${d455_cam_depth} ${d455_cam_width} ${d455_cam_height}"/> -->
+	        <mesh filename="package://realsense2_description/meshes/d455.stl" scale="0.001 0.001 0.001" />
         </geometry>
         <material name="aluminum"/>
