Commit message: Update _d585.urdf.xacro
Updates after new measurements of new model on solid work.
Still need to be updated for every new engineering model.

File: realsense2_description/urdf/_d585.urdf.xacro (robot description, xacro)
@@ -40,9 +40,9 @@
     <xacro:property name="d585_cam_depth" value="0.0931"/>
     <!-- TODO Samer: This parameter is still missing, took it from D455 -->
-    <xacro:property name="d585_cam_mount_from_center_offset" value="0.0377"/> <!-- TODO Samer: check -->
+    <xacro:property name="d585_cam_mount_from_center_offset" value="0.042"/> <!-- TODO Samer: check -->
     <!-- TODO Samer: This parameter is still missing, took it from D455 -->
     <xacro:property name="d585_glass_to_front" value="0.1e-3"/> <!-- TODO Samer: check -->
     <!-- TODO Samer: This parameter is still missing, took it from D455 -->
-    <xacro:property name="d585_zero_depth_to_glass" value="4.55e-3"/> <!-- TODO Samer: check -->
+    <xacro:property name="d585_zero_depth_to_glass" value="0.0056"/> <!-- TODO Samer: check -->
     <!-- TODO Samer: This parameter is still missing, took it from D455 -->
     <xacro:property name="d585_mesh_x_offset" value="${d585_cam_mount_from_center_offset-d585_glass_to_front-d585_zero_depth_to_glass}"/>

Commit message: Update _d585.urdf.xacro

File: realsense2_description/urdf/_d585.urdf.xacro (robot description, xacro)
@@ -39,11 +39,7 @@
     <xacro:property name="d585_cam_height" value="0.043"/>
     <xacro:property name="d585_cam_depth" value="0.0931"/>
-    <!-- TODO Samer: This parameter is still missing, took it from D455 -->
-    <xacro:property name="d585_cam_mount_from_center_offset" value="0.042"/> <!-- TODO Samer: check -->
-    <!-- TODO Samer: This parameter is still missing, took it from D455 -->
-    <xacro:property name="d585_glass_to_front" value="0.1e-3"/> <!-- TODO Samer: check -->
-    <!-- TODO Samer: This parameter is still missing, took it from D455 -->
-    <xacro:property name="d585_zero_depth_to_glass" value="0.0056"/> <!-- TODO Samer: check -->
-    <!-- TODO Samer: This parameter is still missing, took it from D455 -->
+    <xacro:property name="d585_cam_mount_from_center_offset" value="0.042"/> <!-- TODO: Not final numbers, still require refinements -->
+    <xacro:property name="d585_glass_to_front" value="0.1e-3"/> <!-- TODO: Not final numbers, still require refinements -->
+    <xacro:property name="d585_zero_depth_to_glass" value="0.0056"/> <!-- TODO: Not final numbers, still require refinements -->
     <xacro:property name="d585_mesh_x_offset" value="${d585_cam_mount_from_center_offset-d585_glass_to_front-d585_zero_depth_to_glass}"/>
     <!-- The following offset is relative to the physical d585 camera peripherial
@@ -169,7 +165,7 @@
       <link name="${name}_occupancy_optical_frame" />
       <!-- IMU -->
-      <xacro:property name="d585_imu_px" value="0.0114"/> <!-- TODO Samer: check -->
-      <xacro:property name="d585_imu_py" value="-0.0195"/> <!-- TODO Samer: check -->
-      <xacro:property name="d585_imu_pz" value="0"/> <!-- TODO Samer: check -->
+      <xacro:property name="d585_imu_px" value="0.0114"/> <!-- TODO: Not final numbers, still require refinements -->
+      <xacro:property name="d585_imu_py" value="-0.0195"/> <!-- TODO: Not final numbers, still require refinements -->
+      <xacro:property name="d585_imu_pz" value="0"/> <!-- TODO: Not final numbers, still require refinements -->
       <link name="${name}_accel_frame" />
       <link name="${name}_accel_optical_frame" />

Commit message: Fix URDF and LPCL for SC

File: realsense2_description/urdf/_d585.urdf.xacro (robot description, xacro)
@@ -23,5 +23,5 @@
   <xacro:include filename="$(find realsense2_description)/urdf/_materials.urdf.xacro" />
   <xacro:include filename="$(find realsense2_description)/urdf/_usb_plug.urdf.xacro" />
-  <xacro:macro name="sensor_d585" params="parent *origin name:=camera use_nominal_extrinsics:=false">
+  <xacro:macro name="sensor_d585" params="parent *origin name:=camera use_nominal_extrinsics:=false sp_x:=0 sp_y:=0 sp_z:=0 sp_roll:=0 sp_pitch:=0 sp_yaw:=0">
     <xacro:arg name="add_plug" default="false" />
     <xacro:property name="M_PI" value="3.1415926535897931" />
@@ -140,5 +140,5 @@
       <!-- camera labeled point cloud joints and links -->
       <joint name="${name}_labeled_point_cloud_joint" type="fixed">
-        <origin xyz="0 ${d585_cam_depth_to_labeled_point_cloud_offset} 0" rpy="0 0 0" />
+        <origin xyz="${sp_x} ${sp_y} ${sp_z}" rpy="${sp_roll} ${sp_pitch} ${sp_yaw}" />
         <parent link="${name}_link" />
         <child link="${name}_labeled_point_cloud_frame" />
@@ -153,5 +153,5 @@
       <!-- camera occupancy joints and links -->
       <joint name="${name}_occupancy_joint" type="fixed">
-        <origin xyz="0 ${d585_cam_depth_to_labeled_point_cloud_offset} 0" rpy="0 0 0" />
+        <origin xyz="${sp_x} ${sp_y} ${sp_z}" rpy="${sp_roll} ${sp_pitch} ${sp_yaw}" />
         <parent link="${name}_link" />
         <child link="${name}_occupancy_frame" />

File: realsense2_description/urdf/test_d585_camera.urdf.xacro (robot description, xacro)
@@ -3,6 +3,12 @@
   <xacro:arg name="use_nominal_extrinsics" default="false"/>
   <xacro:include filename="$(find realsense2_description)/urdf/_d585.urdf.xacro" />
+  <xacro:arg name="sp_x" default="0.0"/>
+  <xacro:arg name="sp_y" default="0.0"/>
+  <xacro:arg name="sp_z" default="0.0"/>
+  <xacro:arg name="sp_roll" default="0.0"/>
+  <xacro:arg name="sp_pitch" default="0.0"/>
+  <xacro:arg name="sp_yaw" default="0.0"/>
   <link name="base_link" />
-  <xacro:sensor_d585 parent="base_link" use_nominal_extrinsics="$(arg use_nominal_extrinsics)">
+  <xacro:sensor_d585 parent="base_link" use_nominal_extrinsics="$(arg use_nominal_extrinsics)" sp_x="$(arg sp_x)" sp_y="$(arg sp_y)" sp_z="$(arg sp_z)" sp_roll="$(arg sp_roll)" sp_pitch="$(arg sp_pitch)" sp_yaw="$(arg sp_yaw)">
     <origin xyz="0 0 0" rpy="0 0 0"/>
   </xacro:sensor_d585>
